File: Hardware/PCB/detection_board/pm_bias.kicad_sch (KiCad schematic)
At the start: 16 parts, among them J1 Conn_01x01_Socket, J2 Conn_01x01_Socket, U1 MICROFC-60035-SMT-TR1, U2 LT1807, U3 ADCMP601

Commit message: edited schematics
Parts:
- removed J1, J2: Conn_01x01_Socket, Connector_PinSocket_2.54mm:PinSocket_1x01_P2.54mm_Vertical, symbol Connector:Conn_01x01_Socket
- added C5: 10n, symbol Device:C
- added C6: 100n, symbol Device:C
- added JP1: Jumper_2_Small_Bridged, symbol Jumper:Jumper_2_Small_Bridged
- added R8: 30, symbol Device:R
- added R9: 10k, symbol Device:R
Connections:
- net +3V3: now also C5.1, C6.1
- net GND: now also C5.2, C6.2, R9.2
- net comparator_out: now also R8.2; no longer U3.1
- net pm_out: now also JP1.2 (B), R9.1; no longer R4.2
- new net: JP1.1 (A), R4.2
- new net: R8.1, U3.1
Other:
- company: (none) -> UMD Nearspace Balloon Payload Program
- moved on the sheet: C1, C2, C3, C4, R1, R2, R3, R4, R5, R6, R7, U1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
