File: Hardware/PCB/detection_board/detection_board.kicad_sch (KiCad schematic)
At the start: 1 part, among them J1 DE9_Socket_MountingHoles

Commit message: pcb design
Parts:
- added D1, D2, D3: LED, LED_SMD:LED_0805_2012Metric, symbol Device:LED
- added Q1: MMBT3904, Package_TO_SOT_SMD:SOT-23, symbol Transistor_BJT:MMBT3904
- added R10: 60, Resistor_SMD:R_0805_2012Metric, symbol Device:R
- added R11: 1400, Resistor_SMD:R_0805_2012Metric, symbol Device:R
- added R12: 40, Resistor_SMD:R_0805_2012Metric, symbol Device:R
- added R13: 500, Resistor_SMD:R_0805_2012Metric, symbol Device:R
Connections:
- net GND_C is gone; now on net GND: J1.SH (PAD)
- net +3V3: now also J1.3, R10.1, R12.2; no longer J1.2
- net -30V: now also J1.9, D1.1 (K); no longer J1.1
- net GND: now also J1.5, D2.1 (K), Q1.2 (E), R11.2; no longer J1.6
- net comparator_out: now also J1.4; no longer J1.8
- net comparator_ret: now also J1.8; no longer J1.4
- net detection_out: now also J1.2, R13.2; no longer J1.9
- net detection_ret: now also J1.7; no longer J1.5
- net switch_dig: now also J1.1; no longer J1.7
- net switch_ret: now also J1.6; no longer J1.3
- new net: D1.2 (A), R11.1
- new net: Q1.1 (B), R13.1
- new net: D2.2 (A), R10.2
- new net: D3.1 (K), Q1.3 (C)
- new net: D3.2 (A), R12.1

Commit message: board update
Parts:
- removed Q1: MMBT3904, Package_TO_SOT_SMD:SOT-23, symbol Transistor_BJT:MMBT3904
- added Q1: BSS138, Package_TO_SOT_SMD:SOT-23, symbol Transistor_FET:BSS138
- R12: value 40 -> 60
- R13: value 500 -> 10k
Connections:
- net +3V3: now also R12.1; no longer R12.2
- net GND: now also R13.2, Q1.2 (S)
- net detection_out: no longer R13.2
- net switch_dig: now also R13.1, Q1.1 (G)
- net at D3.1 (K): now also R12.2
- net at D3.2 (A): now also Q1.3 (D); no longer R12.1

Commit message: board update
Parts:
- added H1, H2, H3, H4: MountingHole, MountingHole:MountingHole_2.2mm_M2_DIN965_Pad, symbol Mechanical:MountingHole
- added JP1, JP2, JP3: Jumper_2_Small_Bridged, TestPoint:TestPoint_2Pads_Pitch2.54mm_Drill0.8mm, symbol Jumper:Jumper_2_Small_Bridged
- J1: footprint Connector_Dsub:DSUB-9_Pins_Horizontal_P2.77x2.84mm_EdgePinOffset4.94mm_Housed_MountingHolesOffset4.94mm -> D09P33E4GL00LF:AMPHENOL_D09P33E4GL00LF
- R1: renamed from R13; footprint Resistor_SMD:R_0805_2012Metric -> Resistor_SMD:R_0603_1608Metric
- R2: renamed from R12; footprint Resistor_SMD:R_0805_2012Metric -> Resistor_SMD:R_0603_1608Metric
- R3: renamed from R10; footprint Resistor_SMD:R_0805_2012Metric -> Resistor_SMD:R_0603_1608Metric
- R4: renamed from R11; footprint Resistor_SMD:R_0805_2012Metric -> Resistor_SMD:R_0603_1608Metric
- renumbered D1 to -30V_PG1, D2 to 3V3_PG1, D3 to D1
Connections:
- net +3V3: now also JP1.2 (B), JP2.2 (B); no longer R2.1, R3.1
- net -30V: now also JP3.2 (B); no longer -30V_PG1.1 (K)
- new net: -30V_PG1.1 (K), JP3.1 (A)
- new net: JP1.1 (A), R2.1
- new net: JP2.1 (A), R3.1
