File: Hardware/PCB/detection_board/peak_detect.kicad_sch (KiCad schematic)
At the start: 9 parts, among them U1 ${SIM.PARAMS}, U2 ${SIM.PARAMS}, U3 ADG417BN

Commit message: m
Parts:
- removed R1: R, symbol Device:R
- added R301: R, symbol Device:R
- renumbered C2 to C301, C3 to C302, C1 to C303, C4 to C304, D1 to D301, U1 to U301, U3 to U302, U2 to U303
Connections:
- net GND: now also R301.1
- net at U302.1: now also R301.2
Changed lines of the file:
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@@
 		(on_board yes)
 		(dnp no)
-		(property "Reference" "C4"
+		(property "Reference" "C304"
 			(at 172.72 83.82 0)
 			(effects
@@
 			(project ""
 				(path "/871ea243-9d20-4c93-850f-9fe294f22536/0ec79d7b-5798-4abd-9d80-52c9ef728fe7"
-					(reference "C4")
+					(reference "C304")
+					(unit 1)
+				)
+			)
+		)
+	)
+	(symbol
+		(lib_id "Device:R")
+		(at 146.05 113.03 90)
+		(unit 1)
+		(exclude_from_sim no)
+		(in_bom yes)
+		(on_board yes)
+		(dnp no)
+		(property "Reference" "R301"
+			(at 146.05 107.95 90)
+			(effects
+				(font
+					(size 1.27 1.27)
+				)
+			)
+		)
+		(property "Value" "R"
+			(at 146.05 110.49 90)
+			(effects
+				(font
+					(size 1.27 1.27)
+				)
+			)
+		)
+		(property "Footprint" ""
+			(at 146.05 114.808 90)
+			(effects
+				(font
+					(size 1.27 1.27)
+				)
+				(hide yes)
+			)
+		)
+		(property "Datasheet" "~"
+			(at 146.05 113.03 0)
+			(effects
+				(font
+					(size 1.27 1.27)
+				)
+				(hide yes)
+			)
+		)
+		(property "Description" "Resistor"
+			(at 146.05 113.03 0)
+			(effects
+				(font
+					(size 1.27 1.27)
+				)
+				(hide yes)
+			)
+		)
+		(pin "1"
+		)
+		(pin "2"
+		)
+		(instances
+			(project ""
+				(path "/871ea243-9d20-4c93-850f-9fe294f22536/0ec79d7b-5798-4abd-9d80-52c9ef728fe7"
+					(reference "R301")
 					(unit 1)
 				)
@@
 		(on_board yes)
 		(dnp no)
-		(property "Reference" "#PWR07"
+		(property "Reference" "#PWR0304"
 			(at 111.76 95.25 0)
 			(effects
@@
 			(project ""
 				(path "/871ea243-9d20-4c93-850f-9fe294f22536/0ec79d7b-5798-4abd-9d80-52c9ef728fe7"
-					(reference "#PWR07")
+					(reference "#PWR0304")
 					(unit 1)
 				)
@@
 		(on_board yes)
 		(dnp no)
-		(property "Reference" "#PWR05"
+		(property "Reference" "#PWR0301"
 			(at 99.06 95.25 0)
 			(effects
@@
 			(project ""
 				(path "/871ea243-9d20-4c93-850f-9fe294f22536/0ec79d7b-5798-4abd-9d80-52c9ef728fe7"
-					(reference "#PWR05")
+					(reference "#PWR0301")
 					(unit 1)
 				)
@@
 		(dnp no)
 		(fields_autoplaced yes)
-		(property "Reference" "D1"
+		(property "Reference" "D301"
 			(at 118.4275 95.25 0)
 			(effects
@@
 			(project ""
 				(path "/871ea243-9d20-4c93-850f-9fe294f22536/0ec79d7b-5798-4abd-9d80-52c9ef728fe7"
-					(reference "D1")
+					(reference "D301")
 					(unit 1)
 				)
@@
 		(on_board yes)
 		(dnp no)
-		(property "Reference" "C1"
+		(property "Reference" "C303"
 			(at 132.08 106.68 0)
 			(effects
@@
 			(project ""
 				(path "/871ea243-9d20-4c93-850f-9fe294f22536/0ec79d7b-5798-4abd-9d80-52c9ef728fe7"
-					(reference "C1")
+					(reference "C303")
 					(unit 1)
 				)
@@
 		(dnp no)
 		(fields_autoplaced yes)
-		(property "Reference" "#PWR04"
+		(property "Reference" "#PWR0307"
 			(at 182.88 121.92 0)
 			(effects
@@
 			(project ""
 				(path "/871ea243-9d20-4c93-850f-9fe294f22536/0ec79d7b-5798-4abd-9d80-52c9ef728fe7"
-					(reference "#PWR04")
+					(reference "#PWR0307")
 					(unit 1)
 				)
@@
 		(on_board yes)
 		(dnp no)
-		(property "Reference" "C2"
+		(property "Reference" "C301"
 			(at 92.71 83.82 0)
 			(effects
@@
 			(project ""
 				(path "/871ea243-9d20-4c93-850f-9fe294f22536/0ec79d7b-5798-4abd-9d80-52c9ef728fe7"
-					(reference "C2")
-					(unit 1)
-				)
-			)
-		)
-	)
-	(symbol
-		(lib_id "Device:R")
-		(at 146.05 113.03 90)
-		(unit 1)
-		(exclude_from_sim no)
-		(in_bom yes)
-		(on_board yes)
-		(dnp no)
-		(property "Reference" "R1"
-			(at 146.05 107.95 90)
-			(effects
-				(font
-					(size 1.27 1.27)
-				)
-			)
-		)
-		(property "Value" "R"
-			(at 146.05 110.49 90)
-			(effects
-				(font
-					(size 1.27 1.27)
-				)
-			)
-		)
-		(property "Footprint" ""
-			(at 146.05 114.808 90)
-			(effects
-				(font
-					(size 1.27 1.27)
-				)
-				(hide yes)
-			)
-		)
-		(property "Datasheet" "~"
-			(at 146.05 113.03 0)
-			(effects
-				(font
-					(size 1.27 1.27)
-				)
-				(hide yes)
-			)
-		)
-		(property "Description" "Resistor"
-			(at 146.05 113.03 0)
-			(effects
-				(font
-					(size 1.27 1.27)
-				)
-				(hide yes)
-			)
-		)
-		(pin "2"
-		)
-		(pin "1"
-		)
-		(instances
-			(project ""
-				(path "/871ea243-9d20-4c93-850f-9fe294f22536/0ec79d7b-5798-4abd-9d80-52c9ef728fe7"
-					(reference "R1")
+					(reference "C301")
 					(unit 1)
 				)
@@
 		(dnp no)
 		(fields_autoplaced yes)
-		(property "Reference" "#PWR01"
+		(property "Reference" "#PWR0302"
 			(at 104.14 76.2 0)
 			(effects
@@
 			(project ""
 				(path "/871ea243-9d20-4c93-850f-9fe294f22536/0ec79d7b-5798-4abd-9d80-52c9ef728fe7"
-					(reference "#PWR01")
+					(reference "#PWR0302")
 					(unit 1)
 				)
@@
 		(on_board yes)
 		(dnp no)
-		(property "Reference" "#PWR06"
+		(property "Reference" "#PWR0306"
 			(at 175.26 95.25 0)
 			(effects
@@
 			(project ""
 				(path "/871ea243-9d20-4c93-850f-9fe294f22536/0ec79d7b-5798-4abd-9d80-52c9ef728fe7"
-					(reference "#PWR06")
+					(reference "#PWR0306")
 					(unit 1)
 				)
@@
 		(on_board yes)
 		(dnp no)
-		(property "Reference" "U2"
+		(property "Reference" "U303"
 			(at 189.23 96.52 0)
 			(effects
@@
 			(project ""
 				(path "/871ea243-9d20-4c93-850f-9fe294f22536/0ec79d7b-5798-4abd-9d80-52c9ef728fe7"
-					(reference "U2")
+					(reference "U303")
 					(unit 1)
 				)
@@
 		(dnp no)
 		(fields_autoplaced yes)
-		(property "Reference" "C3"
+		(property "Reference" "C302"
 			(at 111.76 83.8199 0)
 			(effects
@@
 			(project ""
 				(path "/871ea243-9d20-4c93-850f-9fe294f22536/0ec79d7b-5798-4abd-9d80-52c9ef728fe7"
-					(reference "C3")
+					(reference "C302")
 					(unit 1)
 				)
@@
 		(dnp no)
 		(fields_autoplaced yes)
-		(property "Reference" "#PWR03"
+		(property "Reference" "#PWR0305"
 			(at 137.16 121.92 0)
 			(effects
@@
 			(project ""
 				(path "/871ea243-9d20-4c93-850f-9fe294f22536/0ec79d7b-5798-4abd-9d80-52c9ef728fe7"
-					(reference "#PWR03")
+					(reference "#PWR0305")
 					(unit 1)
 				)
@@
 		(on_board yes)
 		(dnp no)
-		(property "Reference" "U1"
+		(property "Reference" "U301"
 			(at 109.22 96.52 0)
 			(effects
@@
 			(project ""
 				(path "/871ea243-9d20-4c93-850f-9fe294f22536/0ec79d7b-5798-4abd-9d80-52c9ef728fe7"
-					(reference "U1")
+					(reference "U301")
 					(unit 1)
 				)
@@
 		(on_board yes)
 		(dnp no)
-		(property "Reference" "U3"
+		(property "Reference" "U302"
 			(at 149.86 101.6 90)
 			(effects
@@
 			(project ""
 				(path "/871ea243-9d20-4c93-850f-9fe294f22536/0ec79d7b-5798-4abd-9d80-52c9ef728fe7"
-					(reference "U3")
+					(reference "U302")
 					(unit 1)
 				)
@@
 		(dnp no)
 		(fields_autoplaced yes)
-		(property "Reference" "#PWR02"
+		(property "Reference" "#PWR0303"
 			(at 104.14 121.92 0)
 			(effects
@@
 			(project ""
 				(path "/871ea243-9d20-4c93-850f-9fe294f22536/0ec79d7b-5798-4abd-9d80-52c9ef728fe7"
-					(reference "#PWR02")
-					(unit 1)
-				)
+					(reference "#PWR0303")
+					(unit 1)
+				)

Commit message: finished schem
Parts:
- removed U301, U303: ${SIM.PARAMS}, symbol Simulation_SPICE:OPAMP
- removed U302: ADG417BN, Package_DIP:DIP-8_W7.62mm, symbol Analog_Switch:ADG417BN
- added C305: 22p, Capacitor_SMD:C_0805_2012Metric, symbol Device:C
- added D302: D_Schottky, Diode_SMD:D_0805_2012Metric, symbol Device:D_Schottky
- added R302: 1k, Resistor_SMD:R_0805_2012Metric, symbol Device:R
- added U2: (no value), Package_SO:SOIC-8_3.9x4.9mm_P1.27mm, symbol New_Library:LT1807
- added U3: TS12A4514DBVR, TS12A4514DBVR:SOT95P280X145-5N, symbol TS12A4514DBVR:TS12A4514DBVR
- added U5: (no value), Package_TO_SOT_SMD:SOT-23-5_HandSoldering, symbol New_Library:OPA365AIDBVT
- C00: renamed from C302; value C -> 10n; footprint (none) -> Capacitor_SMD:C_0805_2012Metric
- C301: value C -> 100n; footprint (none) -> Capacitor_SMD:C_0805_2012Metric
- C303: value C -> 1n; footprint (none) -> Capacitor_SMD:C_0805_2012Metric
- C304: value C -> 10n; footprint (none) -> Capacitor_SMD:C_0805_2012Metric
- D301: footprint (none) -> Diode_SMD:D_0805_2012Metric
- R301: value R -> 50; footprint (none) -> Resistor_SMD:R_0805_2012Metric
Connections:
- net GND: now also U2.4 (V-), U3.1 (COM), U3.3 (GND), U5.2 (V-); no longer R301.1
- net detection_out: now also R302.2, U5.1, U5.4 (-)
- net pm_in: now also U2.5 (+)
- net switch_dig: now also U3.4 (IN)
- net at R301.2: now also C303.1, D301.1 (K), U5.3 (+)
- net at D301.2 (A): now also C305.1, D302.2 (A), U2.7
- net +5V renamed +3V3
- net +3V3: now also U2.8 (V+), U3.5 (V+), U5.5 (V+)
- new net: C305.2, D302.1 (K), R302.1, U2.6 (-)
- new net: R301.1, U3.2 (NO)
Other:
- moved on the sheet: D301

Commit message: Layout changes
Parts:
- U2: value (none) -> LT1807
- U4: renamed from U5; value (none) -> OPA365
- renumbered C00 to C302, C305 to C303, C303 to C304, C304 to C305, R302 to R301, R301 to R302, U3 to U5
Changed lines of the file:
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@@
 		(dnp no)
 		(fields_autoplaced yes)
-		(property "Reference" "U5"
+		(property "Reference" "U4"
 			(at 201.93 97.7198 0)
 			(show_name no)
@@
 			)
 		)
-		(property "Value" ""
+		(property "Value" "OPA365"
 			(at 182.88 101.6 0)
+			(hide yes)
 			(show_name no)
 			(do_not_autoplace no)
@@
 			(project "detection_board"
 				(path "/871ea243-9d20-4c93-850f-9fe294f22536/0ec79d7b-5798-4abd-9d80-52c9ef728fe7"
-					(reference "U5")
+					(reference "U4")
 					(unit 1)
 				)
@@
 		(in_pos_files yes)
 		(dnp no)
-		(property "Reference" "C304"
+		(property "Reference" "C305"
 			(at 172.72 83.82 0)
 			(show_name no)
@@
 			(project "detection_board"
 				(path "/871ea243-9d20-4c93-850f-9fe294f22536/0ec79d7b-5798-4abd-9d80-52c9ef728fe7"
-					(reference "C304")
+					(reference "C305")
 					(unit 1)
 				)
@@
 		(in_pos_files yes)
 		(dnp no)
-		(property "Reference" "C305"
+		(property "Reference" "C303"
 			(at 106.68 106.68 0)
 			(show_name no)
@@
 			(project "detection_board"
 				(path "/871ea243-9d20-4c93-850f-9fe294f22536/0ec79d7b-5798-4abd-9d80-52c9ef728fe7"
-					(reference "C305")
+					(reference "C303")
 					(unit 1)
 				)
@@
 		(in_pos_files yes)
 		(dnp no)
-		(property "Reference" "C303"
+		(property "Reference" "C304"
 			(at 132.08 106.68 0)
 			(show_name no)
@@
 			(project "detection_board"
 				(path "/871ea243-9d20-4c93-850f-9fe294f22536/0ec79d7b-5798-4abd-9d80-52c9ef728fe7"
-					(reference "C303")
+					(reference "C304")
 					(unit 1)
 				)
@@
 			)
 		)
-		(property "Value" ""
+		(property "Value" "LT1807"
 			(at 105.41 101.6 0)
 			(show_name no)
@@
 		(in_pos_files yes)
 		(dnp no)
-		(property "Reference" "R301"
+		(property "Reference" "R302"
 			(at 144.78 105.41 90)
 			(show_name no)
@@
 			(project "detection_board"
 				(path "/871ea243-9d20-4c93-850f-9fe294f22536/0ec79d7b-5798-4abd-9d80-52c9ef728fe7"
-					(reference "R301")
+					(reference "R302")
 					(unit 1)
 				)
@@
 		(dnp no)
 		(fields_autoplaced yes)
-		(property "Reference" "U3"
+		(property "Reference" "U5"
 			(at 179.07 119.38 0)
 			(show_name no)
@@
 			(project "detection_board"
 				(path "/871ea243-9d20-4c93-850f-9fe294f22536/0ec79d7b-5798-4abd-9d80-52c9ef728fe7"
-					(reference "U3")
+					(reference "U5")
 					(unit 1)
 				)
@@
 		(dnp no)
 		(fields_autoplaced yes)
-		(property "Reference" "C00"
+		(property "Reference" "C302"
 			(at 111.76 83.8199 0)
 			(show_name no)
@@
 			(project "detection_board"
 				(path "/871ea243-9d20-4c93-850f-9fe294f22536/0ec79d7b-5798-4abd-9d80-52c9ef728fe7"
-					(reference "C00")
+					(reference "C302")
 					(unit 1)
 				)
@@
 		(in_pos_files yes)
 		(dnp no)
-		(property "Reference" "R302"
+		(property "Reference" "R301"
 			(at 129.54 111.76 90)
 			(show_name no)
@@
 			(project "detection_board"
 				(path "/871ea243-9d20-4c93-850f-9fe294f22536/0ec79d7b-5798-4abd-9d80-52c9ef728fe7"
-					(reference "R302")
-					(unit 1)
-				)
+					(reference "R301")
+					(unit 1)
+				)

Commit message: edited schematics
Parts:
- removed C301: 100n, Capacitor_SMD:C_0805_2012Metric, symbol Device:C
- added C306: 100n, symbol Device:C
- added R300: 10k, symbol Device:R
Connections:
- net +3V3: now also C306.1
- net GND: now also C306.2, R300.2
- net pm_in: now also R300.1
Other:
- company: (none) -> UMD Nearspace Balloon Payload Program
- moved on the sheet: C302, C303, C304, C305, D301, D302, R301, R302, U2B, U4, U5

Commit message: board layout
Parts:
- C306: footprint (none) -> Capacitor_SMD:C_0805_2012Metric
- R300: footprint (none) -> Resistor_SMD:R_0805_2012Metric
Other:
- moved on the sheet: C302, C303, C304, C305, C306, D301, D302, R300, R301, R302, U2B, U4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

Commit message: Board layout
Other:
- moved on the sheet: C302, C303, C304, C305, C306, D301, D302, R300, R301, R302, U2B, U4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

Commit message: pcb design
Parts:
- C302, C303, C304, C305, C306: footprint Capacitor_SMD:C_0805_2012Metric -> Capacitor_SMD:C_0201_0603Metric
- D301, D302: footprint Diode_SMD:D_0805_2012Metric -> Diode_SMD:D_0201_0603Metric
- R300, R301, R302: footprint Resistor_SMD:R_0805_2012Metric -> Resistor_SMD:R_0201_0603Metric
Changed lines of the file:
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@@
 			)
 		)
-		(property "Footprint" "Capacitor_SMD:C_0805_2012Metric"
+		(property "Footprint" "Capacitor_SMD:C_0201_0603Metric"
 			(at 213.0552 121.92 0)
 			(hide yes)
@@
 			)
 		)
-		(property "Footprint" "Capacitor_SMD:C_0805_2012Metric"
+		(property "Footprint" "Capacitor_SMD:C_0201_0603Metric"
 			(at 187.0202 70.485 0)
 			(hide yes)
@@
 			)
 		)
-		(property "Footprint" "Diode_SMD:D_0805_2012Metric"
+		(property "Footprint" "Diode_SMD:D_0201_0603Metric"
 			(at 120.015 86.36 0)
 			(hide yes)
@@
 			)
 		)
-		(property "Footprint" "Capacitor_SMD:C_0805_2012Metric"
+		(property "Footprint" "Capacitor_SMD:C_0201_0603Metric"
 			(at 112.0902 90.17 0)
 			(hide yes)
@@
 			)
 		)
-		(property "Footprint" "Diode_SMD:D_0805_2012Metric"
+		(property "Footprint" "Diode_SMD:D_0201_0603Metric"
 			(at 131.445 81.28 0)
 			(hide yes)
@@
 			)
 		)
-		(property "Footprint" "Capacitor_SMD:C_0805_2012Metric"
+		(property "Footprint" "Capacitor_SMD:C_0201_0603Metric"
 			(at 149.5552 91.44 0)
 			(hide yes)
@@
 			)
 		)
-		(property "Footprint" "Resistor_SMD:R_0805_2012Metric"
+		(property "Footprint" "Resistor_SMD:R_0201_0603Metric"
 			(at 70.612 82.55 90)
 			(hide yes)
@@
 			)
 		)
-		(property "Footprint" "Resistor_SMD:R_0805_2012Metric"
+		(property "Footprint" "Resistor_SMD:R_0201_0603Metric"
 			(at 165.608 86.995 90)
 			(hide yes)
@@
 			)
 		)
-		(property "Footprint" "Capacitor_SMD:C_0805_2012Metric"
+		(property "Footprint" "Capacitor_SMD:C_0201_0603Metric"
 			(at 94.9452 67.945 0)
 			(hide yes)
@@
 			)
 		)
-		(property "Footprint" "Resistor_SMD:R_0805_2012Metric"
+		(property "Footprint" "Resistor_SMD:R_0201_0603Metric"
 			(at 133.35 98.298 90)
 			(hide yes)
