File: Hardware/PCB/detection_board/peak_detect.kicad_sch (KiCad schematic)
At the start: 13 parts, among them U2 LT1807, U4 OPA365, U5 TS12A4514DBVR

Commit message: board update
Parts:
- removed D301, D302: D_Schottky, Diode_SMD:D_0201_0603Metric, symbol Device:D_Schottky
- added D2: BAT54A, Package_TO_SOT_SMD:SOT-23, symbol Diode:BAT54A
- added R18: R, Resistor_SMD:R_0603_1608Metric, symbol Device:R
- C10: renamed from C305; footprint Capacitor_SMD:C_0201_0603Metric -> Capacitor_SMD:C_0603_1608Metric
- C11: renamed from C306; footprint Capacitor_SMD:C_0201_0603Metric -> Capacitor_SMD:C_0603_1608Metric
- C7: renamed from C302; footprint Capacitor_SMD:C_0201_0603Metric -> Capacitor_SMD:C_0603_1608Metric
- C8: renamed from C303; footprint Capacitor_SMD:C_0201_0603Metric -> Capacitor_SMD:C_0603_1608Metric
- C9: renamed from C304; footprint Capacitor_SMD:C_0201_0603Metric -> Capacitor_SMD:C_0603_1608Metric
- R15: renamed from R300; footprint Resistor_SMD:R_0201_0603Metric -> Resistor_SMD:R_0603_1608Metric
- R16: renamed from R301; footprint Resistor_SMD:R_0201_0603Metric -> Resistor_SMD:R_0603_1608Metric
- R17: renamed from R302; footprint Resistor_SMD:R_0201_0603Metric -> Resistor_SMD:R_0603_1608Metric
Connections:
- net detection_out: now also R18.2; no longer R16.2, U4.1, U4.4 (-)
- net at C9.1, R17.2, U4.3 (+): now also D2.2
- net at C8.2, R16.1, U2.6 (-): now also D2.1
- net at C8.1, U2.7: now also D2.3
- new net: R16.2, R18.1, U4.1, U4.4 (-)
