File: Hardware/PCB/detection_board/detection_board.kicad_pcb (KiCad board)
At the start: 2 copper layers, 26 parts, among them J1 Screw_Terminal_01x01, U1 MICROFC-60035-SMT-TR1, U3 TS12A4514DBVR

Commit message: Layout changes
Parts:
- added J2: Conn_01x01_Socket, Connector_PinSocket_2.54mm:PinSocket_1x01_P2.54mm_Vertical, F.Cu at (139.6, 95.3)
- added J3: Conn_01x01_Socket, Connector_PinSocket_2.54mm:PinSocket_1x01_P2.54mm_Vertical, F.Cu at (133.0, 90.8)
- added J4: Conn_01x01_Socket, Connector_PinSocket_2.54mm:PinSocket_1x01_P2.54mm_Vertical, F.Cu at (133.0, 95.3)
- added J5: Conn_01x01_Socket, Connector_PinSocket_2.54mm:PinSocket_1x01_P2.54mm_Vertical, F.Cu at (133.0, 99.9)
- J1: value Screw_Terminal_01x01 -> Conn_01x01_Socket; footprint TerminalBlock_MetzConnect:TerminalBlock_MetzConnect_360271_1x01_Horizontal_ScrewM3.0_Boxed -> Connector_PinSocket_2.54mm:PinSocket_1x01_P2.54mm_Vertical
- U2: value ~ -> LT1807
- U3: renamed from U4; value ~ -> ADCMP601
- U4: renamed from U5; value ~ -> OPA365
- moved J1 53.5 mm to (139.6, 90.8)
- moved R6 4.54 mm to (113.8, 72.2)
- moved R301 3.94 mm to (148.9, 63.6)
- moved D302 2.66 mm to (142.8, 63.2)
- moved R5 2.47 mm to (115.9, 68.9)
- moved U2 2.39 mm to (133.6, 51.5)
- moved U4 0.96 mm to (144.2, 51.7)
- moved R302 0.89 mm to (147.3, 57.9)
- moved C302 0.36 mm to (137.8, 57.2)
- renumbered C2 to C1, C3 to C2, C4 to C3, C00 to C302, C305 to C303, C303 to C304, C304 to C305, C1 to C4, R3 to R1, R4 to R2, R2 to R3, R302 to R301, R301 to R302, R1 to R4, U3 to U5
Connections:
- J1 pad 1: switch_dig -> -30V

Commit message: Created PCB design
Created PCB design
yerp
Parts:
- U1: moved to B.Cu
- moved R1 60.3 mm to (167.0, 99.0)
- moved J4 58.6 mm to (191.5, 92.0)
- moved R2 56.8 mm to (171.1, 87.5)
- moved C1 51.7 mm to (167.5, 95.0)
- moved C2 48.0 mm to (167.5, 89.5)
- moved U5 47.6 mm to (190.2, 81.0)
- moved C305 47.2 mm to (184.6, 61.5)
- moved U4 46.7 mm to (189.5, 63.0)
- moved U1 46.3 mm to (168.0, 77.5), turned to 180 degrees
- moved C3 45.6 mm to (167.6, 83.5)
- moved J5 45.2 mm to (177.5, 92.0)
- moved R6 43.0 mm to (154.0, 87.5)
- moved R7 42.8 mm to (160.4, 83.0)
- moved C304 42.3 mm to (179.5, 70.0)
- moved R302 41.6 mm to (187.0, 70.5)
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Other:
- board outline added: 60 x 50 mm
- board text added: "Brandon B, Anirudh C, Larry T, Sarah T, Prachi W"
- board text added: "Electra 2027 Rev 3"

Commit message: 2
Parts:
- removed C301: 100n, Capacitor_SMD:C_0805_2012Metric
- removed J2, J3, J4, J5: Conn_01x01_Socket, Connector_PinSocket_2.54mm:PinSocket_1x01_P2.54mm_Vertical
- added C306: 100n, Capacitor_SMD:C_0805_2012Metric, F.Cu at (188.8, 53.4)
- added C5: 10n, Capacitor_SMD:C_0805_2012Metric, F.Cu at (165.9, 84.6)
- added C6: 100n, Capacitor_SMD:C_0805_2012Metric, F.Cu at (167.0, 51.5)
- added JP1: Jumper_2_Small_Bridged, TestPoint:TestPoint_2Pads_Pitch2.54mm_Drill0.8mm, F.Cu at (171.1, 83.9)
- added R300: 10k, Resistor_SMD:R_0805_2012Metric, F.Cu at (161.9, 76.8)
- added R8: 30, Resistor_SMD:R_0805_2012Metric, F.Cu at (160.5, 57.7)
- added R9: 10k, Resistor_SMD:R_0805_2012Metric, F.Cu at (169.1, 86.8)
- J1: value Conn_01x01_Socket -> DE9_Pins; footprint Connector_PinSocket_2.54mm:PinSocket_1x01_P2.54mm_Vertical -> Connector_Dsub:DSUB-9_Pins_Horizontal_P2.77x2.84mm_EdgePinOffset4.94mm_Housed_MountingHolesOffset4.94mm
- moved C305 43.6 mm to (153.2, 91.8), turned to -90 degrees
- moved U4 42.0 mm to (157.0, 89.7), turned to 180 degrees
- moved U5 42.0 mm to (149.6, 91.7)
- moved R302 39.9 mm to (149.8, 84.9)
- moved R5 34.8 mm to (171.8, 52.1)
- moved R6 34.8 mm to (171.8, 57.6)
- moved U3 31.2 mm to (169.9, 45.9)
- moved R1 28.1 mm to (157.6, 72.5), turned to -90 degrees
- moved C1 27.8 mm to (158.5, 68.7)
- moved R7 25.9 mm to (167.8, 58.1)
- moved R301 25.3 mm to (152.9, 82.0), turned to -90 degrees
- moved R4 25.1 mm to (174.2, 82.4), turned to -90 degrees
- moved C304 24.2 mm to (161.4, 86.0), turned to -90 degrees
- moved C2 23.7 mm to (162.1, 66.5)
- moved D301 20.2 mm to (158.0, 83.9), turned to 90 degrees
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Connections:
- J1 pad 1: -30V -> GND
- R4 pad 2: /peak_detect/pm_in -> Net-(JP1-A)
- U3 pad 1: comparator_out -> Net-(R8-Pad1)
Routing:
- net +3V3: track 0.00 -> 12.3 mm
- net /peak_detect/pm_in: track 0.00 -> 6.59 mm
- net Net-(U2A--): track 0.00 -> 5.46 mm

Commit message: Board layout
Parts:
- removed C302: 10n, Capacitor_SMD:C_0805_2012Metric
- removed C306: 100n, Capacitor_SMD:C_0805_2012Metric
- moved U3 44.0 mm to (171.0, 89.9)
- moved R5 37.9 mm to (180.2, 89.0), turned to -90 degrees
- moved C6 37.6 mm to (174.7, 88.3)
- moved R6 36.4 mm to (181.0, 92.8)
- moved R7 34.7 mm to (175.7, 91.9), turned to -90 degrees
- moved R8 32.7 mm to (165.6, 90.0), turned to -90 degrees
- moved C4 31.1 mm to (176.2, 77.9)
- moved R3 31.0 mm to (177.1, 81.3)
- moved R1 21.5 mm to (179.1, 73.7), turned to 0 degrees
- moved C1 17.0 mm to (175.0, 72.9), turned to -90 degrees
- moved R2 8.18 mm to (170.8, 73.4), turned to 180 degrees
- moved C2 7.76 mm to (167.0, 72.5), turned to -90 degrees
- moved R9 5.20 mm to (168.2, 91.9), turned to -90 degrees
- moved C3 3.77 mm to (163.1, 72.6)
- moved R302 3.65 mm to (152.5, 87.3)
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Routing:
- net +3V3: track 12.3 -> 0.00 mm
- net /peak_detect/pm_in: track 6.59 -> 13.6 mm
- net Net-(U2A--): track 5.46 -> 0.00 mm
Other:
- board text added: "Electra 2027 Rev 3 Detection Board"
- board text removed: "Electra 2027 Rev 3"

Commit message: board edit
Parts:
- added C302: 10n, Capacitor_SMD:C_0805_2012Metric, F.Cu at (152.5, 115.7)
- added C306: 100n, Capacitor_SMD:C_0805_2012Metric, F.Cu at (152.5, 118.7)
- added REF**: MountingHole_2.2mm_M2_DIN965_Pad, MountingHole:MountingHole_2.2mm_M2_DIN965_Pad, F.Cu at (141.3, 101.7)
- added REF**: MountingHole_2.2mm_M2_DIN965_Pad, MountingHole:MountingHole_2.2mm_M2_DIN965_Pad, F.Cu at (194.6, 101.8)
- added REF**: MountingHole_2.2mm_M2_DIN965_Pad, MountingHole:MountingHole_2.2mm_M2_DIN965_Pad, F.Cu at (141.3, 58.2)
- added REF**: MountingHole_2.2mm_M2_DIN965_Pad, MountingHole:MountingHole_2.2mm_M2_DIN965_Pad, F.Cu at (194.6, 58.4)
- J1: value DE9_Pins -> DE9_Socket_MountingHoles
- moved J1 1.46 mm to (161.2, 97.0)
Connections:
- J1 pad 1: GND -> -30V
- J1 pad 2: GND -> +3V3
- J1 pad 4: +3V3 -> GND
- J1 pad 5: -30V -> GND
- J1 pad 6: detection_out -> GND
- J1 pad 7: comparator_out -> switch_dig
- J1 pad 8: switch_dig -> comparator_out
- J1 pad 9: GND -> detection_out
Other:
- outline, holes or cut-outs redrawn

Commit message: pcb design
Parts:
- added D1: LED, LED_SMD:LED_0805_2012Metric, F.Cu at (157.1, 70.5)
- added D2: LED, LED_SMD:LED_0805_2012Metric, F.Cu at (150.5, 70.5)
- added D3: LED, LED_SMD:LED_0805_2012Metric, F.Cu at (144.5, 92.0)
- added Q1: MMBT3904, Package_TO_SOT_SMD:SOT-23, F.Cu at (145.1, 85.0)
- added R10: 60, Resistor_SMD:R_0805_2012Metric, F.Cu at (150.5, 74.0)
- added R11: 1400, Resistor_SMD:R_0805_2012Metric, F.Cu at (157.1, 74.0)
- added R12: 40, Resistor_SMD:R_0805_2012Metric, F.Cu at (151.1, 90.5)
- added R13: 500, Resistor_SMD:R_0805_2012Metric, F.Cu at (147.0, 79.5)
- added TP1: TestPoint, TestPoint:TestPoint_Pad_1.5x1.5mm, F.Cu at (180.0, 87.0)
- added TP2: TestPoint, TestPoint:TestPoint_Pad_1.5x1.5mm, F.Cu at (180.0, 90.5)
- C1, C2, C3, C302, C303, C304, C305, C306, C4, C5, C6: footprint Capacitor_SMD:C_0805_2012Metric -> Capacitor_SMD:C_0201_0603Metric
- D301, D302: footprint Diode_SMD:D_0805_2012Metric -> Diode_SMD:D_0201_0603Metric
- R1, R2, R3, R300, R301, R302, R4, R5, R6, R7, R8, R9: footprint Resistor_SMD:R_0805_2012Metric -> Resistor_SMD:R_0201_0603Metric
- moved C306 36.5 mm to (155.8, 82.3)
- moved C302 34.6 mm to (166.5, 84.0), turned to -90 degrees
- moved R6 15.0 mm to (166.5, 88.7), turned to 90 degrees
- moved R5 12.2 mm to (168.0, 89.3), turned to 90 degrees
- moved U5 9.99 mm to (152.7, 83.5)
- moved R302 7.72 mm to (156.2, 80.5)
- moved R8 7.67 mm to (173.0, 91.8)
- moved R1 7.57 mm to (171.7, 75.0)
- moved R301 7.38 mm to (161.2, 80.0), turned to 180 degrees
- moved R7 7.08 mm to (169.0, 89.7)
- moved D301 6.94 mm to (164.7, 81.8), turned to 0 degrees
- moved C305 6.67 mm to (158.5, 86.3)
- moved U4 6.01 mm to (159.7, 83.5)
- moved C6 5.59 mm to (170.2, 91.5)
- moved C1 5.36 mm to (170.0, 74.8)
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Connections:
- J1 pad 1: -30V -> switch_dig
- J1 pad 2: +3V3 -> detection_out
- J1 pad 3: GND -> +3V3
- J1 pad 4: GND -> comparator_out
- J1 pad 7: switch_dig -> GND
- J1 pad 8: comparator_out -> GND
- J1 pad 9: detection_out -> -30V
- J1 pad SH: GND_C -> GND
Routing:
- net +3V3: track 0.00 -> 75.5 mm, vias 0 -> 4
- net -30V: track 0.00 -> 64.0 mm
- net detection_out: track 0.00 -> 35.9 mm
- net GND: track 0.11 -> 29.9 mm, vias 0 -> 85
- net switch_dig: track 0.00 -> 15.5 mm
- net Net-(JP1-A): track 0.00 -> 11.1 mm
- net Net-(U5-NO): track 0.00 -> 10.4 mm
- net Net-(D301-K): track 0.00 -> 9.48 mm, vias 0 -> 2
- net Net-(U2A--): track 0.00 -> 8.22 mm, vias 0 -> 1
- net Net-(D3-K): track 0.00 -> 6.68 mm
- net Net-(C4-Pad2): track 0.00 -> 6.47 mm
- net comparator_out: track 0.00 -> 6.23 mm
- net Net-(D302-K): track 0.00 -> 5.82 mm
- net Net-(C2-Pad2): track 0.00 -> 5.43 mm, vias 0 -> 1
- net Net-(D3-A): track 0.00 -> 5.36 mm
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- added copper zone on B.Cu, net GND
- added copper zone on F.Cu, net GND

Commit message: board update
Parts:
- removed REF** (x4): MountingHole_2.2mm_M2_DIN965_Pad, MountingHole:MountingHole_2.2mm_M2_DIN965_Pad
- Q1: value MMBT3904 -> BSS138
- R12: value 40 -> 60
- R13: value 500 -> 10k
- moved R13 2.18 mm to (144.9, 80.2), turned to 180 degrees
- moved R12 1.56 mm to (149.5, 90.5), turned to 180 degrees
- moved D3 0.48 mm to (144.4, 91.5), turned to 90 degrees
- moved Q1 0.11 mm to (145.0, 84.9)
Connections:
- Q1 pad 1: Net-(Q1-B) -> switch_dig
- Q1 pad 3: Net-(D3-K) -> Net-(D3-A)
- R12 pad 1: Net-(D3-A) -> +3V3
- R12 pad 2: +3V3 -> Net-(D3-K)
- R13 pad 1: Net-(Q1-B) -> switch_dig
- R13 pad 2: detection_out -> GND
Routing:
- net switch_dig: track 15.5 -> 29.5 mm
- net detection_out: track 35.9 -> 22.7 mm
- net Net-(Q1-B): track 4.60 -> 0.00 mm
- net GND: track 29.9 -> 33.5 mm, vias 85 -> 99
- net Net-(D2-A): track 3.50 -> 5.20 mm
- net Net-(D3-K): track 6.68 -> 5.08 mm
- net +3V3: track 75.5 -> 77.1 mm

Commit message: nn
Parts:
- removed JP1: Jumper_2_Small_Bridged, TestPoint:TestPoint_2Pads_Pitch2.54mm_Drill0.8mm
- added SW1: SW_SPST, Connector_PinHeader_2.54mm:PinHeader_1x03_P2.54mm_Vertical, F.Cu at (169.4, 86.0)
- moved R3 1.51 mm to (174.0, 81.3), turned to -90 degrees
- moved C4 0.96 mm to (175.0, 81.3), turned to -90 degrees
- moved R4 0.81 mm to (174.0, 82.8)
Routing:
- net Net-(C4-Pad2): track 6.47 -> 4.51 mm
- net Net-(U2A--): track 8.22 -> 6.75 mm
- net GND: track 33.5 -> 32.6 mm, vias 99 -> 114
- net Net-(SW1-A): track 11.1 -> 11.8 mm
