File: Hardware/PCB/detection_board/detection_board.kicad_pcb (KiCad board)
At the start: 2 copper layers, 60 x 50 mm, 42 parts, among them J1 DE9_Socket_MountingHoles, Q1 BSS138, SW1 SW_SPST, U1 MICROFC-60035-SMT-TR1, U2 LT1807, U3 ADCMP601, U4 OPA365, U5 TS12A4514DBVR

Commit message: board update
Parts:
- removed D301, D302: D_Schottky, Diode_SMD:D_0201_0603Metric
- removed SW1: SW_SPST, Connector_PinHeader_2.54mm:PinHeader_1x03_P2.54mm_Vertical
- removed TP2: TestPoint, TestPoint:TestPoint_Pad_1.5x1.5mm
- added D2: BAT54A, Package_TO_SOT_SMD:SOT-23, F.Cu at (161.7, 77.4)
- added H1: MountingHole, MountingHole:MountingHole_2.2mm_M2_DIN965_Pad, F.Cu at (194.2, 58.8)
- added H2: MountingHole, MountingHole:MountingHole_2.2mm_M2_DIN965_Pad, F.Cu at (141.2, 101.8)
- added H3: MountingHole, MountingHole:MountingHole_2.2mm_M2_DIN965_Pad, F.Cu at (141.8, 58.8)
- added H4: MountingHole, MountingHole:MountingHole_2.2mm_M2_DIN965_Pad, F.Cu at (194.2, 101.2)
- added JP1: Jumper_2_Small_Bridged, TestPoint:TestPoint_2Pads_Pitch2.54mm_Drill0.8mm, F.Cu at (149.1, 88.2)
- added JP2: Jumper_2_Small_Bridged, TestPoint:TestPoint_2Pads_Pitch2.54mm_Drill0.8mm, F.Cu at (148.2, 74.0)
- added JP3: Jumper_2_Small_Bridged, TestPoint:TestPoint_2Pads_Pitch2.54mm_Drill0.8mm, F.Cu at (160.6, 67.9)
- added R12: 0, Resistor_SMD:R_0603_1608Metric, F.Cu at (171.7, 81.4)
- added R18: R, Resistor_SMD:R_0603_1608Metric, F.Cu at (160.3, 84.6)
- C1: renamed from C3; footprint Capacitor_SMD:C_0201_0603Metric -> Capacitor_SMD:C_0603_1608Metric
- C10: renamed from C305; footprint Capacitor_SMD:C_0201_0603Metric -> Capacitor_SMD:C_0603_1608Metric
- C11: renamed from C306; footprint Capacitor_SMD:C_0201_0603Metric -> Capacitor_SMD:C_0603_1608Metric
- C2, C6: footprint Capacitor_SMD:C_0201_0603Metric -> Capacitor_SMD:C_0603_1608Metric
- C3: renamed from C1; footprint Capacitor_SMD:C_0201_0603Metric -> Capacitor_SMD:C_0603_1608Metric
- C4: renamed from C5; footprint Capacitor_SMD:C_0201_0603Metric -> Capacitor_SMD:C_0603_1608Metric
- C5: renamed from C4; footprint Capacitor_SMD:C_0201_0603Metric -> Capacitor_SMD:C_0603_1608Metric
- C7: renamed from C302; footprint Capacitor_SMD:C_0201_0603Metric -> Capacitor_SMD:C_0603_1608Metric
- C8: renamed from C303; footprint Capacitor_SMD:C_0201_0603Metric -> Capacitor_SMD:C_0603_1608Metric
- C9: renamed from C304; footprint Capacitor_SMD:C_0201_0603Metric -> Capacitor_SMD:C_0603_1608Metric
- J1: footprint Connector_Dsub:DSUB-9_Pins_Horizontal_P2.77x2.84mm_EdgePinOffset4.94mm_Housed_MountingHolesOffset4.94mm -> D09P33E4GL00LF:AMPHENOL_D09P33E4GL00LF
- R1: renamed from R13; footprint Resistor_SMD:R_0805_2012Metric -> Resistor_SMD:R_0603_1608Metric
- R10: renamed from R6; footprint Resistor_SMD:R_0201_0603Metric -> Resistor_SMD:R_0603_1608Metric
- R11: renamed from R9; footprint Resistor_SMD:R_0201_0603Metric -> Resistor_SMD:R_0603_1608Metric
- R13: renamed from R7; footprint Resistor_SMD:R_0201_0603Metric -> Resistor_SMD:R_0603_1608Metric
- R14: renamed from R8; footprint Resistor_SMD:R_0201_0603Metric -> Resistor_SMD:R_0603_1608Metric
- R15: renamed from R300; footprint Resistor_SMD:R_0201_0603Metric -> Resistor_SMD:R_0603_1608Metric
- R16: renamed from R301; footprint Resistor_SMD:R_0201_0603Metric -> Resistor_SMD:R_0603_1608Metric
- R17: renamed from R302; footprint Resistor_SMD:R_0201_0603Metric -> Resistor_SMD:R_0603_1608Metric
- R2: renamed from R12; footprint Resistor_SMD:R_0805_2012Metric -> Resistor_SMD:R_0603_1608Metric
- R3: renamed from R10; footprint Resistor_SMD:R_0805_2012Metric -> Resistor_SMD:R_0603_1608Metric
- R4: renamed from R11; footprint Resistor_SMD:R_0805_2012Metric -> Resistor_SMD:R_0603_1608Metric
- R5: renamed from R2; footprint Resistor_SMD:R_0201_0603Metric -> Resistor_SMD:R_0603_1608Metric
- R6: renamed from R1; footprint Resistor_SMD:R_0201_0603Metric -> Resistor_SMD:R_0603_1608Metric
- R7: renamed from R3; footprint Resistor_SMD:R_0201_0603Metric -> Resistor_SMD:R_0603_1608Metric
- R8: renamed from R4; footprint Resistor_SMD:R_0201_0603Metric -> Resistor_SMD:R_0603_1608Metric
- R9: renamed from R5; footprint Resistor_SMD:R_0201_0603Metric -> Resistor_SMD:R_0603_1608Metric
- TP1: value TestPoint -> pm_out
- moved R17 8.24 mm to (148.9, 76.5)
- moved C11 8.03 mm to (148.8, 78.4), turned to 180 degrees
- moved C10 6.64 mm to (153.5, 82.0), turned to 180 degrees
- moved R11 6.08 mm to (171.7, 83.0), turned to 0 degrees
- moved J1 5.64 mm to (166.7, 95.8)
- moved R16 5.59 mm to (156.2, 77.4), turned to -90 degrees
- moved R15 5.18 mm to (161.8, 74.4), turned to 180 degrees
- moved U5 4.91 mm to (148.3, 81.3)
- moved C3 4.31 mm to (169.1, 70.6)
- moved R10 4.16 mm to (163.9, 85.4)
- moved 3V3_PG1 3.95 mm to (148.4, 67.2)
- moved R3 3.78 mm to (148.5, 70.8)
- moved C1 3.62 mm to (162.7, 72.0)
- moved -30V_PG1 3.45 mm to (156.0, 67.2)
- moved R4 3.45 mm to (156.1, 70.7)
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- renumbered D1 to -30V_PG1, D2 to 3V3_PG1, D3 to D1
Connections:
- -30V_PG1 pad 1: -30V -> Net-(-30V_PG1-K)
- R16 pad 2: detection_out -> Net-(U4--)
- R2 pad 1: +3V3 -> Net-(JP1-A)
- R3 pad 1: +3V3 -> Net-(JP2-A)
- U4 pad 1: detection_out -> Net-(U4--)
- U4 pad 4: detection_out -> Net-(U4--)
Routing:
- net detection_out: track 22.7 -> 10.5 mm
- net Net-(U4--): track 0.00 -> 7.34 mm
- net Net-(U2B--): track 5.82 -> 13.0 mm
- net Net-(U4-+): track 9.48 -> 16.0 mm
- net +3V3: track 77.1 -> 82.1 mm
- net GND: track 32.6 -> 36.8 mm, vias 114 -> 160
- net Net-(-30V_PG1-K): track 0.00 -> 3.91 mm
- net -30V: track 64.0 -> 60.1 mm
- net Net-(JP2-A): track 0.00 -> 3.83 mm
- net Net-(U5-NO): track 10.4 -> 6.70 mm
- net Net-(R12-Pad1): track 11.8 -> 8.85 mm
- net Net-(U3--): track 3.89 -> 5.96 mm
- net Net-(JP1-A): track 0.00 -> 2.05 mm
- net switch_dig: track 29.5 -> 31.5 mm
- net Net-(C3-Pad2): track 2.54 -> 4.26 mm
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