File: Hardware/PCB/monitorMain/Teensy-Sensor_Board/Teensy-Sensor_Board.kicad_pcb (KiCad board)
At the start: 2 copper layers, 83.5 x 132 mm, 17 parts, among them J1 DE9_Pins, J2 DA15_Pins, J3 Screw_Terminal_01x02, U1 LD1117V33, U2 LD1117V33, U3 LM7805_TO220, U4 DEV-16771, U5 COSEL_MUW30515C

Commit message: board update
Parts:
- J1: footprint Connector_Dsub:DSUB-9_Pins_Horizontal_P2.77x2.84mm_EdgePinOffset9.90mm_Housed_MountingHolesOffset11.32mm -> D09P33E4GL00LF:AMPHENOL_D09P33E4GL00LF
- moved J1 6.69 mm to (142.9, 35.3)
Routing:
- net Net-(ADT7410-Pins1-Pin_1): track 139.8 -> 143.3 mm
- net Net-(U5--Vout): track 25.8 -> 28.1 mm
